Commit message: Updated nega-max and arduino code

File: robot_arm/robot_arm.urdf (robot description, URDF)
Before this commit: robot robot_arm, 10 links, 9 joints
Links:
- link base_link: mass 1.0 -> None; geometry collision mesh filename=Base.STL scale=1 1 1; visual mesh filename=Base.STL scale=1 1 1
